File: Schaltplan/221110_Schaltplan/221110_Schaltplan.kicad_pcb (KiCad board)
At the start: 2 copper layers, 27 parts, among them J0 LDR0, J1 LDR1, J10 LDR2, J11 LDR3, J12 V_solar, J13 V_solar, J14 Dspl GND, J15 Dspl Vcc, J16 Mode Button GND, J17 Poti GND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

Commit message: Finish Schaltplan
Parts:
- moved J4 1.02 mm to (174.0, 100.6)
- moved J5 1.02 mm to (176.5, 100.6)
Routing:
- net Net-(A0-Pad29): track 33.0 -> 297.1 mm
- net Net-(A0-Pad26): track 0.00 -> 5.90 mm
- net Net-(A0-Pad28): track 0.00 -> 5.90 mm
- net Net-(A0-Pad27): track 0.00 -> 5.90 mm
- net Net-(A0-Pad25): track 0.00 -> 5.90 mm
- net Net-(A0-Pad14): track 48.2 -> 47.2 mm
- net Net-(A0-Pad13): track 48.2 -> 47.2 mm
Other:
- board outline added: 81.3 x 83.8 mm
