File: Schaltplan/221110_Schaltplan/221110_Schaltplan.kicad_sch (KiCad schematic)
At the start: 22 parts, among them J0 LDR0, J1 LDR1, J10 LDR2, J11 LDR3, J12 V_solar, J13 V_solar, J14 Dspl GND, J15 Dspl Vcc, J2 LDR2, J3 LDR3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

Commit message: Add Connector for Mode Button and Poti
Parts:
- added J16: Mode Button GND, symbol Connector:Conn_01x01_Female
- added J17: Poti GND, symbol Connector:Conn_01x01_Female
- added J18: Mode Button, symbol Connector:Conn_01x01_Female
- added J19: Poti 5V, symbol Connector:Conn_01x01_Female
- added J20: Poti, symbol Connector:Conn_01x01_Female
Connections:
- net at A0.5 (+5V), J15.1 (Pin_1), J6.2 (Pin_2)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: now also J19.1 (Pin_1)
- net at A0.29 (GND), J0.1 (Pin_1), J1.1 (Pin_1)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: now also J16.1 (Pin_1), J17.1 (Pin_1)
- net at U0.6 (CH5): now also J20.1 (Pin_1)
- net at A0.23 (D8): now also J18.1 (Pin_1)
Changed lines of the file:
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@@
   (junction (at 113.03 99.06) (diameter 0) (color 0 0 0 0)
   )
+  (junction (at 133.35 99.06) (diameter 0) (color 0 0 0 0)
+  )
   (junction (at 138.43 30.48) (diameter 0) (color 0 0 0 0)
   )
@@
   (junction (at 123.19 99.06) (diameter 0) (color 0 0 0 0)
   )
+  (junction (at 66.04 31.75) (diameter 0) (color 0 0 0 0)
+  )
   (junction (at 128.27 99.06) (diameter 0) (color 0 0 0 0)
   )
+  (junction (at 138.43 99.06) (diameter 0) (color 0 0 0 0)
+  )
   (junction (at 66.04 34.29) (diameter 0) (color 0 0 0 0)
   )
@@
     (stroke (width 0) (type default) (color 0 0 0 0))
   )
+  (wire (pts (xy 133.35 99.06) (xy 138.43 99.06))
+    (stroke (width 0) (type default) (color 0 0 0 0))
+  )
   (wire (pts (xy 102.87 30.48) (xy 138.43 30.48))
     (stroke (width 0) (type default) (color 0 0 0 0))
@@
     (stroke (width 0) (type default) (color 0 0 0 0))
   )
+  (wire (pts (xy 110.49 66.04) (xy 101.6 66.04))
+    (stroke (width 0) (type default) (color 0 0 0 0))
+  )
   (wire (pts (xy 58.42 44.45) (xy 66.04 44.45))
     (stroke (width 0) (type default) (color 0 0 0 0))
@@
     (stroke (width 0) (type default) (color 0 0 0 0))
   )
+  (wire (pts (xy 138.43 99.06) (xy 143.51 99.06))
+    (stroke (width 0) (type default) (color 0 0 0 0))
+  )
   (wire (pts (xy 38.1 57.15) (xy 38.1 69.85))
     (stroke (width 0) (type default) (color 0 0 0 0))
@@
     (stroke (width 0) (type default) (color 0 0 0 0))
   )
+  (wire (pts (xy 101.6 66.04) (xy 101.6 49.53))
+    (stroke (width 0) (type default) (color 0 0 0 0))
+  )
   (wire (pts (xy 139.7 76.2) (xy 139.7 80.01))
     (stroke (width 0) (type default) (color 0 0 0 0))
@@
     (stroke (width 0) (type default) (color 0 0 0 0))
   )
-  (wire (pts (xy 135.89 66.04) (xy 139.7 66.04))
-    (stroke (width 0) (type default) (color 0 0 0 0))
-  )
   (wire (pts (xy 49.53 52.07) (xy 40.64 52.07))
     (stroke (width 0) (type default) (color 0 0 0 0))
@@
     (stroke (width 0) (type default) (color 0 0 0 0))
   )
-  (wire (pts (xy 135.89 63.5) (xy 139.7 63.5))
+  (wire (pts (xy 35.56 26.67) (xy 66.04 26.67))
     (stroke (width 0) (type default) (color 0 0 0 0))
   )
@@
     (stroke (width 0) (type default) (color 0 0 0 0))
   )
+  (wire (pts (xy 101.6 49.53) (xy 97.79 49.53))
+    (stroke (width 0) (type default) (color 0 0 0 0))
+  )
   (wire (pts (xy 66.04 82.55) (xy 66.04 88.9))
     (stroke (width 0) (type default) (color 0 0 0 0))
@@
     (stroke (width 0) (type default) (color 0 0 0 0))
   )
-  (wire (pts (xy 135.89 68.58) (xy 139.7 68.58))
-    (stroke (width 0) (type default) (color 0 0 0 0))
-  )
   (wire (pts (xy 135.89 76.2) (xy 139.7 76.2))
     (stroke (width 0) (type default) (color 0 0 0 0))
@@
     (stroke (width 0) (type default) (color 0 0 0 0))
   )
+  (wire (pts (xy 66.04 26.67) (xy 66.04 31.75))
+    (stroke (width 0) (type default) (color 0 0 0 0))
+  )
   (wire (pts (xy 86.36 71.12) (xy 110.49 71.12))
     (stroke (width 0) (type default) (color 0 0 0 0))
@@
     (stroke (width 0) (type default) (color 0 0 0 0))
   )
+  (wire (pts (xy 35.56 72.39) (xy 55.88 72.39))
+    (stroke (width 0) (type default) (color 0 0 0 0))
+  )
   (wire (pts (xy 58.42 44.45) (xy 58.42 46.99))
     (stroke (width 0) (type default) (color 0 0 0 0))
@@
   (wire (pts (xy 86.36 67.31) (xy 95.25 67.31))
     (stroke (width 0) (type default) (color 0 0 0 0))
+  )
+  (symbol (lib_id "Connector:Conn_01x01_Female") (at 30.48 72.39 0) (mirror y) (unit 1)
+    (in_bom yes) (on_board yes)
+    (property "Reference" "J20" (id 0) (at 26.67 71.12 0))
+    (property "Value" "Poti" (id 1) (at 26.67 73.66 0))
+    (property "Footprint" "" (id 2) (at 30.48 72.39 0)
+      (effects (font (size 1.27 1.27)) hide)
+    )
+    (property "Datasheet" "~" (id 3) (at 30.48 72.39 0)
+      (effects (font (size 1.27 1.27)) hide)
+    )
+    (pin "1")
   )
   (symbol (lib_id "Connector:Conn_01x03_Male") (at 143.51 25.4 0) (mirror y) (unit 1)
@@
     (pin "1")
   )
+  (symbol (lib_id "Connector:Conn_01x01_Female") (at 30.48 26.67 0) (mirror y) (unit 1)
+    (in_bom yes) (on_board yes)
+    (property "Reference" "J19" (id 0) (at 26.67 25.4 0))
+    (property "Value" "Poti 5V" (id 1) (at 26.67 27.94 0))
+    (property "Footprint" "" (id 2) (at 30.48 26.67 0)
+      (effects (font (size 1.27 1.27)) hide)
+    )
+    (property "Datasheet" "~" (id 3) (at 30.48 26.67 0)
+      (effects (font (size 1.27 1.27)) hide)
+    )
+    (pin "1")
+  )
   (symbol (lib_id "Connector:Conn_01x01_Female") (at 30.48 46.99 0) (mirror y) (unit 1)
     (in_bom yes) (on_board yes) (fields_autoplaced)
@@
     (pin "1")
   )
+  (symbol (lib_id "Connector:Conn_01x01_Female") (at 138.43 104.14 90) (mirror x) (unit 1)
+    (in_bom yes) (on_board yes)
+    (property "Reference" "J16" (id 0) (at 137.16 107.95 0)
+      (effects (font (size 1.27 1.27)) (justify right))
+    )
+    (property "Value" "Mode Button GND" (id 1) (at 139.7 116.84 0)
+      (effects (font (size 1.27 1.27)) (justify right))
+    )
+    (property "Footprint" "" (id 2) (at 138.43 104.14 0)
+      (effects (font (size 1.27 1.27)) hide)
+    )
+    (property "Datasheet" "~" (id 3) (at 138.43 104.14 0)
+      (effects (font (size 1.27 1.27)) hide)
+    )
+    (pin "1")
+  )
   (symbol (lib_id "Connector:Conn_01x01_Female") (at 133.35 104.14 90) (mirror x) (unit 1)
     (in_bom yes) (on_board yes)
@@
     (pin "1")
     (pin "2")
+  )
+  (symbol (lib_id "Connector:Conn_01x01_Female") (at 92.71 49.53 0) (mirror y) (unit 1)
+    (in_bom yes) (on_board yes) (fields_autoplaced)
+    (property "Reference" "J18" (id 0) (at 93.345 44.45 0))
+    (property "Value" "Mode Button" (id 1) (at 93.345 46.99 0))
+    (property "Footprint" "" (id 2) (at 92.71 49.53 0)
+      (effects (font (size 1.27 1.27)) hide)
+    )
+    (property "Datasheet" "~" (id 3) (at 92.71 49.53 0)
+      (effects (font (size 1.27 1.27)) hide)
+    )
+    (pin "1")
   )
   (symbol (lib_id "Connector:Conn_01x03_Male") (at 160.02 25.4 0) (mirror y) (unit 1)
@@
     (pin "1")
   )
+  (symbol (lib_id "Connector:Conn_01x01_Female") (at 143.51 104.14 90) (mirror x) (unit 1)
+    (in_bom yes) (on_board yes)
+    (property "Reference" "J17" (id 0) (at 142.24 107.95 0)
+      (effects (font (size 1.27 1.27)) (justify right))
+    )
+    (property "Value" "Poti GND" (id 1) (at 144.78 113.03 0)
+      (effects (font (size 1.27 1.27)) (justify right))
+    )
+    (property "Footprint" "" (id 2) (at 143.51 104.14 0)
+      (effects (font (size 1.27 1.27)) hide)
+    )
+    (property "Datasheet" "~" (id 3) (at 143.51 104.14 0)
+      (effects (font (size 1.27 1.27)) hide)
+    )
+    (pin "1")
+  )
   (symbol (lib_id "Connector:Conn_01x01_Female") (at 144.78 80.01 0) (unit 1)
-    (in_bom yes) (on_board yes) (fields_autoplaced)
+    (in_bom yes) (on_board yes)
     (property "Reference" "J5" (id 0) (at 146.05 78.7399 0)
       (effects (font (size 1.27 1.27)) (justify left))
@@
       (reference "J15") (unit 1) (value "Dspl Vcc") (footprint "")
     )
+    (path "/8f57826e-eab5-4fcf-b280-2ee4fbec2d1f"
+      (reference "J16") (unit 1) (value "Mode Button GND") (footprint "")
+    )
+    (path "/ea43efc2-2c8c-489d-bf80-23fcf9a49960"
+      (reference "J17") (unit 1) (value "Poti GND") (footprint "")
+    )
+    (path "/af7625e2-d367-4613-a1f3-49cfbe4bc67c"
+      (reference "J18") (unit 1) (value "Mode Button") (footprint "")
+    )
+    (path "/4bb16671-a089-49bc-85ad-d9d4691be964"
+      (reference "J19") (unit 1) (value "Poti 5V") (footprint "")
+    )
+    (path "/16e7a555-a5af-456f-9493-bc8f926d27a8"
+      (reference "J20") (unit 1) (value "Poti") (footprint "")
+    )
     (path "/23832a94-6b8b-4745-9f1f-2ed2d107749d"

Commit message: Add Footprints to Schematic
Parts:
- J0, J1, J10, J11, J12, J13, J14, J15, J16, J17, J18, J19, J2, J20, J3, J4, J5, J8, J9: footprint (none) -> Connector_PinHeader_2.54mm:PinHeader_1x01_P2.54mm_Vertical
- J6, J7: footprint (none) -> Connector_PinHeader_2.54mm:PinHeader_1x03_P2.54mm_Vertical
- R? (x4): footprint (none) -> Resistor_THT:R_Axial_DIN0207_L6.3mm_D2.5mm_P10.16mm_Horizontal

Commit message: Add PCB
Parts:
- gave numbers to parts that had none: 4
Changed lines of the file:
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@@
   (symbol (lib_id "Device:R") (at 53.34 36.83 270) (mirror x) (unit 1)
     (in_bom yes) (on_board yes)
-    (property "Reference" "R?" (id 0) (at 53.34 34.29 90))
+    (property "Reference" "R1" (id 0) (at 53.34 34.29 90))
     (property "Value" "10k" (id 1) (at 53.34 36.83 90))
     (property "Footprint" "Resistor_THT:R_Axial_DIN0207_L6.3mm_D2.5mm_P10.16mm_Horizontal" (id 2) (at 53.34 38.608 90)
@@
   (symbol (lib_id "Device:R") (at 53.34 41.91 270) (mirror x) (unit 1)
     (in_bom yes) (on_board yes)
-    (property "Reference" "R?" (id 0) (at 53.34 39.37 90))
+    (property "Reference" "R2" (id 0) (at 53.34 39.37 90))
     (property "Value" "10k" (id 1) (at 53.34 41.91 90))
     (property "Footprint" "Resistor_THT:R_Axial_DIN0207_L6.3mm_D2.5mm_P10.16mm_Horizontal" (id 2) (at 53.34 43.688 90)
@@
   (symbol (lib_id "Device:R") (at 53.34 46.99 270) (mirror x) (unit 1)
     (in_bom yes) (on_board yes)
-    (property "Reference" "R?" (id 0) (at 53.34 44.45 90))
+    (property "Reference" "R3" (id 0) (at 53.34 44.45 90))
     (property "Value" "10k" (id 1) (at 53.34 46.99 90))
     (property "Footprint" "Resistor_THT:R_Axial_DIN0207_L6.3mm_D2.5mm_P10.16mm_Horizontal" (id 2) (at 53.34 48.768 90)
@@
   (symbol (lib_id "Device:R") (at 53.34 52.07 270) (mirror x) (unit 1)
     (in_bom yes) (on_board yes)
-    (property "Reference" "R?" (id 0) (at 53.34 49.53 90))
+    (property "Reference" "R4" (id 0) (at 53.34 49.53 90))
     (property "Value" "10k" (id 1) (at 53.34 52.07 90))
     (property "Footprint" "Resistor_THT:R_Axial_DIN0207_L6.3mm_D2.5mm_P10.16mm_Horizontal" (id 2) (at 53.34 53.848 90)
@@
     )
     (path "/23832a94-6b8b-4745-9f1f-2ed2d107749d"
-      (reference "R?") (unit 1) (value "10k") (footprint "Resistor_THT:R_Axial_DIN0207_L6.3mm_D2.5mm_P10.16mm_Horizontal")
+      (reference "R1") (unit 1) (value "10k") (footprint "Resistor_THT:R_Axial_DIN0207_L6.3mm_D2.5mm_P10.16mm_Horizontal")
     )
     (path "/7da4a42f-e779-4782-bd86-e6825e2a528c"
-      (reference "R?") (unit 1) (value "10k") (footprint "Resistor_THT:R_Axial_DIN0207_L6.3mm_D2.5mm_P10.16mm_Horizontal")
+      (reference "R2") (unit 1) (value "10k") (footprint "Resistor_THT:R_Axial_DIN0207_L6.3mm_D2.5mm_P10.16mm_Horizontal")
     )
     (path "/7eadc527-4c1e-4236-8a8d-f7e76dc7192e"
-      (reference "R?") (unit 1) (value "10k") (footprint "Resistor_THT:R_Axial_DIN0207_L6.3mm_D2.5mm_P10.16mm_Horizontal")
+      (reference "R3") (unit 1) (value "10k") (footprint "Resistor_THT:R_Axial_DIN0207_L6.3mm_D2.5mm_P10.16mm_Horizontal")
     )
     (path "/ab689dc6-b8fa-4ff8-9f6a-fe9e4b723df3"
-      (reference "R?") (unit 1) (value "10k") (footprint "Resistor_THT:R_Axial_DIN0207_L6.3mm_D2.5mm_P10.16mm_Horizontal")
+      (reference "R4") (unit 1) (value "10k") (footprint "Resistor_THT:R_Axial_DIN0207_L6.3mm_D2.5mm_P10.16mm_Horizontal")
     )
     (path "/3d25220e-19e2-4df3-aa54-dba8597cde77"

Commit message: Change CircuitDiagram to match new CAD Design
Parts:
- removed J6: Srv0, Connector_PinHeader_2.54mm:PinHeader_1x03_P2.54mm_Vertical, symbol Connector:Conn_01x03_Male
- removed J7: Srv1, Connector_PinHeader_2.54mm:PinHeader_1x03_P2.54mm_Vertical, symbol Connector:Conn_01x03_Male
- added J21, J25: GND, Connector_PinHeader_2.54mm:PinHeader_1x01_P2.54mm_Vertical, symbol Connector:Conn_01x01_Female
- added J22: Srv0, Connector_PinHeader_2.54mm:PinHeader_1x03_P2.54mm_Vertical, symbol Connector:Conn_01x03_Male
- added J23: Srv1, Connector_PinHeader_2.54mm:PinHeader_1x03_P2.54mm_Vertical, symbol Connector:Conn_01x03_Male
- added J24: Vextra, Connector_PinHeader_2.54mm:PinHeader_1x01_P2.54mm_Vertical, symbol Connector:Conn_01x01_Female
- added J26: 5V, Connector_PinHeader_2.54mm:PinHeader_1x01_P2.54mm_Vertical, symbol Connector:Conn_01x01_Female
Connections:
- net at A0.20 (D5): now also J22.1 (Pin_1)
- net at A0.5 (+5V), J15.1 (Pin_1), J19.1 (Pin_1)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: now also J26.1 (Pin_1)
- net at A0.29 (GND), J0.1 (Pin_1), J1.1 (Pin_1)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: now also J22.3 (Pin_3), J23.3 (Pin_3)
- net at A0.21 (D6): now also J23.1 (Pin_1)
- net at A0.7 (GND): now also J21.1 (Pin_1), J25.1 (Pin_1)
- new net: J22.2 (Pin_2), J23.2 (Pin_2), J24.1 (Pin_1)
